File: hardware/followMe/followMe.kicad_pcb (KiCad board)
At the start: 2 copper layers, 33 x 17.8 mm, 5 parts, among them J1 FTDI, J2 I2C, J3 Analog, J6 Analog, J7 Digital

Commit message: version 1.00
First Versiyon
Parts:
- added D1: BAV99, Package_TO_SOT_SMD:SOT-23, F.Cu at (164.9, 83.9)
- added D2: BAV99, Package_TO_SOT_SMD:SOT-23, F.Cu at (156.2, 83.9)
- added D5: LED, LED_SMD:LED_1206_3216Metric_Pad1.42x1.75mm_HandSolder, F.Cu at (156.0, 97.7)
- added D6: LED, LED_SMD:LED_1206_3216Metric_Pad1.42x1.75mm_HandSolder, F.Cu at (164.3, 97.7)
- added D7: LED, LED_SMD:LED_1206_3216Metric_Pad1.42x1.75mm_HandSolder, B.Cu at (160.0, 97.7)
- added J4: Vi+, Connector_PinHeader_2.54mm:PinHeader_1x02_P2.54mm_Vertical, F.Cu at (101.9, 57.6)
- added J5: Vi-, Connector_PinHeader_2.54mm:PinHeader_1x02_P2.54mm_Vertical, F.Cu at (106.5, 57.6)
- added J8: Vo-, Connector_PinHeader_2.54mm:PinHeader_1x02_P2.54mm_Vertical, F.Cu at (111.2, 57.6)
- added J9: Vo+, Connector_PinHeader_2.54mm:PinHeader_1x02_P2.54mm_Vertical, F.Cu at (115.8, 57.6)
- added Q1: MMBT2222A, Package_TO_SOT_SMD:SOT-23, F.Cu at (107.3, 78.1)
- added R10: NC, Resistor_SMD:R_0603_1608Metric, F.Cu at (166.1, 93.1)
- added R101: R, Resistor_SMD:R_0805_2012Metric_Pad1.20x1.40mm_HandSolder, F.Cu at (101.9, 63.9)
- added R102: R, Resistor_SMD:R_0805_2012Metric_Pad1.20x1.40mm_HandSolder, F.Cu at (101.9, 66.9)
- added R103: 220, Resistor_SMD:R_0805_2012Metric_Pad1.20x1.40mm_HandSolder, F.Cu at (101.9, 69.8)
- added R104: 220, Resistor_SMD:R_0805_2012Metric_Pad1.20x1.40mm_HandSolder, F.Cu at (101.9, 72.8)
- added R105: 220, Resistor_SMD:R_0805_2012Metric_Pad1.20x1.40mm_HandSolder, F.Cu at (101.9, 75.7)
- added R106: 220, Resistor_SMD:R_0805_2012Metric_Pad1.20x1.40mm_HandSolder, F.Cu at (101.9, 78.7)
- added R107: 4k7, Resistor_SMD:R_0805_2012Metric_Pad1.20x1.40mm_HandSolder, F.Cu at (106.7, 63.9)
- added R108: 4k7, Resistor_SMD:R_0805_2012Metric_Pad1.20x1.40mm_HandSolder, F.Cu at (106.7, 66.9)
- added R109: 4k7, Resistor_SMD:R_0805_2012Metric_Pad1.20x1.40mm_HandSolder, F.Cu at (106.7, 69.8)
- added R110: 4k7, Resistor_SMD:R_0805_2012Metric_Pad1.20x1.40mm_HandSolder, F.Cu at (106.7, 72.8)
- added R2: 1k, Resistor_SMD:R_2010_5025Metric, F.Cu at (160.1, 76.1)
- added R3: NC, Resistor_SMD:R_0603_1608Metric, F.Cu at (157.1, 90.2)
- added R4: R, Resistor_SMD:R_0603_1608Metric, F.Cu at (165.9, 90.2)
- added R5: R, Resistor_SMD:R_0603_1608Metric, F.Cu at (160.0, 90.2)
- added R6: NC, Resistor_SMD:R_0603_1608Metric, F.Cu at (163.0, 90.2)
- added R7: 1k5, Resistor_SMD:R_1206_3216Metric, F.Cu at (156.2, 94.4)
- added R8: NC, Resistor_SMD:R_0603_1608Metric, F.Cu at (154.1, 90.2)
- added R9: NC, Resistor_SMD:R_0603_1608Metric, F.Cu at (164.4, 94.9)
- added TP1: TestPoint, TestPoint:TestPoint_Pad_D1.5mm, B.Cu at (165.7, 73.2)
- added TP2: TestPoint, TestPoint:TestPoint_Pad_D1.5mm, B.Cu at (157.7, 71.8)
- added TP3: TestPoint, TestPoint:TestPoint_Pad_D1.5mm, B.Cu at (154.3, 97.7)
- added TP4: TestPoint, TestPoint:TestPoint_Pad_D1.5mm, B.Cu at (165.7, 97.7)
- added TP5: TestPoint, TestPoint:TestPoint_Pad_D1.5mm, B.Cu at (152.5, 90.2)
Routing:
- net Net-(D7-A): track 0.00 -> 24.8 mm, vias 0 -> 1
- net Net-(D1-A): track 0.00 -> 23.4 mm, vias 0 -> 2
- net Net-(D5-K): track 0.00 -> 21.9 mm, vias 0 -> 1
- net /schineder button led circuit/Vin1: track 0.00 -> 19.8 mm, vias 0 -> 1
- net Net-(D1-K-Pad1): track 0.00 -> 18.4 mm
- net Net-(D5-A): track 0.00 -> 16.6 mm
- net /schineder button led circuit/Vin2: track 0.00 -> 14.1 mm, vias 0 -> 2
- net /schineder button led circuit/Fill: track 0.00 -> 12.6 mm
- net Net-(D6-A): track 0.00 -> 12.2 mm, vias 0 -> 1
- added copper zone on F.Cu, net /schineder button led circuit/Fill
